File: Boost_Buck_Converter.kicad_sch (KiCad schematic)
At the start: 0 parts

Commit message: add boost-buck converter fixed 3.3V, charger battery Li-on 1S, cut-off circuit's supply. modify gitignore
Parts:
- added C1, C2, C3: 10uF 10V, PCM_Capacitor_SMD_AKL:C_0603_1608Metric, symbol PCM_Capacitor_US_AKL:C_0603
- added C4: 0.1uF 10V, PCM_Capacitor_SMD_AKL:C_0603_1608Metric, symbol PCM_Capacitor_US_AKL:C_0603
- added R1: 100R, PCM_Resistor_SMD_AKL:R_0603_1608Metric, symbol PCM_Resistor_US_AKL:R_0603
- added U2: TPS63002DRCR, EasyEDA:VSON-10_L3.0-W3.0-P0.50-BL-EP_TPS62410DRCR, symbol EasyEDA:TPS63002DRCR
- added U3: 2.2uH, EasyEDA:IND-SMD_L7.0-W6.6_MCW-0650-220, symbol EasyEDA:L_7x6.6mm SMD
Connections:
- new net: C4.1, R1.2, U2.6 (EN), U2.7 (PS/SYNC), U2.8 (VINA)
- new net: U2.4 (L1), U3.1
- new net: U2.2 (L2), U3.2
- new net +3V3: C1.1, U2.1 (VOUT), U2.10 (FB)
- new net GND: C1.2, C2.2, C3.2, C4.2, U2.11 (EP), U2.3 (PGND), U2.9 (GND)
- new net VCC: C3.1, R1.1, U2.5 (VIN)
